File: ReceiverRF/receiverKiCad/capteurs.kicad_sch (KiCad schematic)
At the start: 11 parts, among them J1 Conn_Coaxial, J3 Conn_01x04, U4 MLX90393SLW-ABA-011-RE

Commit message: correction mineure, logo Idefix, commande PCBWAY
Parts:
- J1: value Conn_Coaxial -> RF2-03E-T-00-50-G; Digikey (none) -> 2057-RF2-03E-T-00-50-G-ND
- MLX_A0, MLX_A1: value 0 -> jumper
- MLX_C1, MLX_C2: value 100n -> 100nF; Digikey (none) -> 2679-AGC0402X7R500-104KNPTR-ND
- MLX_C3: value 1u -> 1uF; Digikey (none) -> 2679-AGC0603X7R250-105KXPTR-ND
- MLX_R1, MLX_R2: Digikey (none) -> 311-10KJRCT-ND
- RF1: value ~ -> BAT54T1G; Digikey (none) -> BAT54T1GOSCT-ND
- U4: Digikey (none) -> MLX90393SLW-ABA-011-RECT-ND
Changed lines of the file:
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@@
+			)
+		)
+		(property "Digikey" "311-10KJRCT-ND"
+			(at 99.06 71.12 0)
+			(effects
+				(font
+					(size 1.27 1.27)
+				)
+				(hide yes)
 			)
 		)
@@
 			)
 		)
-		(property "Value" "0"
+		(property "Value" "jumper"
 			(at 113.03 59.69 90)
 			(effects
@@
 		)
 		(property "Description" ""
+			(at 110.49 58.42 0)
+			(effects
+				(font
+					(size 1.27 1.27)
+				)
+				(hide yes)
+			)
+		)
+		(property "Digikey" ""
 			(at 110.49 58.42 0)
 			(effects
@@
 			)
 		)
+		(property "Digikey" "311-10KJRCT-ND"
+			(at 110.49 68.58 0)
+			(effects
+				(font
+					(size 1.27 1.27)
+				)
+				(hide yes)
+			)
+		)
 		(pin "1"
 		)
@@
 			)
 		)
-		(property "Value" "100n"
+		(property "Value" "100nF"
 			(at 105.41 36.83 0)
 			(effects
@@
 		)
 		(property "Description" ""
+			(at 102.87 35.56 0)
+			(effects
+				(font
+					(size 1.27 1.27)
+				)
+				(hide yes)
+			)
+		)
+		(property "Digikey" "2679-AGC0402X7R500-104KNPTR-ND"
 			(at 102.87 35.56 0)
 			(effects
@@
 			)
 		)
+		(property "Digikey" "MLX90393SLW-ABA-011-RECT-ND"
+			(at 44.45 52.07 0)
+			(effects
+				(font
+					(size 1.27 1.27)
+				)
+				(hide yes)
+			)
+		)
 		(pin "1"
 		)
@@
 			)
 		)
-		(property "Value" "~"
+		(property "Value" "BAT54T1G"
 			(at 44.45 106.68 0)
 			(effects
@@
 		)
 		(property "Description" ""
+			(at 54.61 107.95 0)
+			(effects
+				(font
+					(size 1.27 1.27)
+				)
+				(hide yes)
+			)
+		)
+		(property "Digikey" "BAT54T1GOSCT-ND"
 			(at 54.61 107.95 0)
 			(effects
@@
 			)
 		)
-		(property "Value" "100n"
+		(property "Value" "100nF"
 			(at 49.53 36.83 0)
 			(effects
@@
 			)
 		)
+		(property "Digikey" "2679-AGC0402X7R500-104KNPTR-ND"
+			(at 46.99 35.56 0)
+			(effects
+				(font
+					(size 1.27 1.27)
+				)
+				(hide yes)
+			)
+		)
 		(pin "1"
 		)
@@
 			)
 		)
-		(property "Value" "1u"
+		(property "Value" "1uF"
 			(at 87.63 36.83 0)
 			(effects
@@
 		)
 		(property "Description" ""
+			(at 85.09 35.56 0)
+			(effects
+				(font
+					(size 1.27 1.27)
+				)
+				(hide yes)
+			)
+		)
+		(property "Digikey" "  2679-AGC0603X7R250-105KXPTR-ND"
 			(at 85.09 35.56 0)
 			(effects
@@
 			)
 		)
-		(property "Value" "0"
+		(property "Value" "jumper"
 			(at 101.6 59.69 90)
 			(effects
@@
 		)
 		(property "Description" ""
+			(at 99.06 58.42 0)
+			(effects
+				(font
+					(size 1.27 1.27)
+				)
+				(hide yes)
+			)
+		)
+		(property "Digikey" ""
 			(at 99.06 58.42 0)
 			(effects
@@
 			)
 		)
+		(property "Digikey" ""
+			(at 39.37 156.21 0)
+			(effects
+				(font
+					(size 1.27 1.27)
+				)
+				(hide yes)
+			)
+		)
 		(pin "1"
 		)
@@
 			)
 		)
-		(property "Value" "Conn_Coaxial"
+		(property "Value" "RF2-03E-T-00-50-G"
 			(at 22.352 104.14 0)
 			(effects
@@
 			(at 25.4 107.95 0)
 			(effects
+				(font
+					(size 1.27 1.27)
+				)
+				(hide yes)
+			)
+		)
+		(property "Digikey" "  2057-RF2-03E-T-00-50-G-ND"
+			(at 25.4 107.95 0)
+			(effects
