File: ReceiverRF/receiverKiCad/receiver.kicad_pcb (KiCad board)
At the start: 2 copper layers, 95.4 x 60 mm, 74 parts, among them J1 Conn_Coaxial, J2 Conn_01x05_Socket, J3 Conn_01x04, Q1 MMBT3904, SW1 SW_Push, SW2 SW_Push, SW3 SW_Push, SW4 SW_Push, SW5 SW_SPST, U1 STM32F103RET6, U2 NCV5501DT33RKG, U3 NJM2882F05-TE1, U4 MLX90393SLW-ABA-011-RE, Y1 Crystal_GND24

Commit message: correction mineure, logo Idefix, commande PCBWAY
Parts:
- added Idéfix le GAULois: LOGO, LOGO, B.Cu at (149.6, 88.3)
- BUZ_D1, RF1: value ~ -> BAT54T1G
- BZ1: value Buzzer -> SMTB-0927-TW-R
- CSTL_C1, CSTL_C2: value 16p -> 16pF
- D1, D2, D3: value vert -> LTST-C170GKT
- FB1: value 120R -> ILBB0603ER121V
- J1: value Conn_Coaxial -> RF2-03E-T-00-50-G
- LED_R1, LED_R2, LED_R3, PWR_R1, PWR_R2, PWR_R3, PWR_R4: value 145 -> 145R
- MLX_A0, MLX_A1: value 0 -> jumper
- MLX_C1, MLX_C2, PWR_C4, STM_C1, STM_C3, STM_C4, STM_C5, S_C10, S_C2: value 100n -> 100nF
- MLX_C3, PWR_C3, STM_C8, STM_C9: value 1u -> 1uF
- PWR_C1, STM_C6: value 10u -> 10uF
- PWR_C2: value 4.7u -> 4.7uF
- PWR_C5, S_C7: value 10n -> 10nF
- PWR_D1, PWR_D2: value Rouge -> LTST-C190EKT
- RV1: value 10k -> RK09K1130A5R
- Y1: value Crystal_GND24 -> YG8M000000S418
Connections:
- U1 pad 50: unconnected-(U1-PA15-Pad50) -> MLX_INT
- U1 pad 51: MLX_INT -> unconnected-(U1-PC10-Pad51)
Routing:
- net GND: track 24.0 -> 23.3 mm, vias 60 -> 66
