File: ReceiverRF/receiverKiCad/receiver.kicad_pcb (KiCad board)
At the start: 2 copper layers, 100 x 116.6 mm, 84 parts, among them J1 RF2-03E-T-00-50-G, J2 Conn_01x05_Socket, J3 Conn_01x02_Socket, J4 Conn_01x04, Q1 MMBT3904, Q2 PMOS, SW1 SW_Push, SW2 SW_Push, SW3 SW_Push, SW4 SW_Push, SW5 SW_SPDT, U1 STM32F103RET6, U2 NCV5501DT33RKG, U3 NJM2882F05-TE1, U4 MLX90393SLW-ABA-011-RE, U5 TXS0102DCUR, Y1 CTX853CT-ND

Commit message: revision schematic before tracing
Parts:
- removed IdéFIX le GAULois: LOGO, LOGO
- PWR_D1: value LTST-C190EKT -> LED_0805_2012Metric
- RF1: value BAT54T1G -> RFM22B
- moved D1 15.4 mm to (147.5, 78.3), turned to 0 degrees
- moved PWR_R5 11.9 mm to (147.5, 75.9), turned to 180 degrees
- moved Q2 11.6 mm to (147.5, 81.5), turned to -90 degrees
- moved SW5 9.82 mm to (139.6, 84.9), turned to 180 degrees
- moved D4 9.72 mm to (141.7, 69.0), turned to 90 degrees
- moved LLS_R2 9.17 mm to (124.4, 123.0)
- moved LLS_C1 9.17 mm to (124.3, 112.1)
- moved LLS_C2 9.17 mm to (124.3, 120.0)
- moved U5 9.17 mm to (124.3, 115.8)
- moved D3 3.27 mm to (138.3, 69.1)
- moved D2 3.27 mm to (135.1, 69.0)
- moved J4 2.73 mm to (112.4, 122.2)
- moved S_R4 0.83 mm to (153.3, 59.3)
- moved STM_C1 0.37 mm to (156.5, 51.1)
Routing:
- net +3.3V: track 0.00 -> 36.2 mm
- net GND: track 0.00 -> 17.8 mm
- net +5V: track 0.00 -> 15.3 mm
- net NRST: track 0.00 -> 11.2 mm
- net /Capteurs/ANT: track 0.00 -> 10.2 mm
- net VCC: track 0.00 -> 9.83 mm
- net OSC_IN: track 2.34 -> 10.2 mm
- net +3.3VA: track 0.00 -> 6.55 mm
- net Net-(MLX_A1-B): track 0.00 -> 6.17 mm
- net Net-(MLX_A0-B): track 0.00 -> 5.67 mm
- net Net-(CSTL_C2-Pad1): track 2.27 -> 6.70 mm
- net Net-(PWR_D2-A): track 0.00 -> 3.57 mm
- net OSC_OUT: track 0.00 -> 3.38 mm
- net Net-(PWR_R3-Pad2): track 0.00 -> 3.34 mm
- net Net-(PWR_R2-Pad2): track 0.00 -> 2.60 mm
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- added copper zone on B.Cu, net GND
