File: ReceiverRF/receiverKiCad/receiver.kicad_sch (KiCad schematic)
At the start: 23 parts, among them J2 Conn_01x05_Socket, U1 STM32F103RET6, Y1 Crystal_GND24

Commit message: correction mineure, logo Idefix, commande PCBWAY
Parts:
- CSTL_C1, CSTL_C2: value 16p -> 16pF; Digikey (none) -> 478-11769-1-ND
- FB1: value 120R -> ILBB0603ER121V; Digikey (none) -> 541-2290-1-ND
- I2C_R1, I2C_R2, STM_R3, S_R1: Digikey (none) -> 311-10KJRCT-ND
- STM_C1, STM_C3, STM_C4, STM_C5, S_C10, S_C2: value 100n -> 100nF; Digikey (none) -> 2679-AGC0402X7R500-104KNPTR-ND
- STM_C6: value 10u -> 10uF; Digikey (none) -> 2679-AGC1206X6S250-106KXETR-ND
- STM_C8, STM_C9: value 1u -> 1uF; Digikey (none) -> 2679-AGC0603X7R250-105KXPTR-ND
- STM_R2: Digikey (none) -> P1.5KDCCT-ND
- S_C7: value 10n -> 10nF; Digikey (none) -> 2679-AGC0402X7R500-103KNPTR-ND
- S_R4: Digikey (none) -> P10.0LCT-ND
- U1: Digikey (none) -> 497-6444-ND
- Y1: value Crystal_GND24 -> YG8M000000S418; Digikey (none) -> 3372-YG8M000000S418TR-ND
Connections:
- net MLX_INT: now also U1.50 (PA15); no longer U1.51 (PC10)
