File: ReceiverRF/receiverKiCad/receiver.kicad_sch (KiCad schematic)
At the start: 24 parts, among them J2 Conn_01x05_Socket, J3 Conn_01x02_Socket, U1 STM32F103RET6, Y1 406C35D08M00000

Commit message: Refactor timer handling and add TRANSMIT/RECEIVE definition macros
Parts:
- J2, J3, JP1: now left out of the parts list
- STM_C6: Digikey 2679-AGC1206X6S250-106KXETR-ND -> 1276-1804-1-ND
- Y1: Digikey CTX853CT-ND -> 110-406C35D08M00000CT-ND
Changed lines of the file:
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@@
 			)
 		)
-		(property "Datasheet" "https://www.st.com/resource/en/datasheet/stm32f103re.pdf"
+		(property "Datasheet" "https://www.digikey.com/en/products/detail/stmicroelectronics/STM32F103RET6/1852094?s=N4IgTCBcDaICwE4DsBaAbHTKByAREAugL5A"
 			(at 153.67 97.79 0)
 			(effects
@@
 			)
 		)
-		(property "Description" ""
+		(property "Description" "Microprocessor"
 			(at 153.67 97.79 0)
 			(effects
@@
 			)
 		)
-		(property "Description" ""
+		(property "Description" "1k5 Res"
 			(at 39.37 93.98 0)
 			(effects
@@
 			)
 		)
-		(property "Description" ""
+		(property "Description" "16pF Cap"
 			(at 46.99 137.16 0)
 			(effects
@@
 			)
 		)
-		(property "Description" ""
+		(property "Description" "10k Res"
 			(at 107.95 54.61 0)
 			(effects
@@
 			)
 		)
-		(property "Description" "120 ohm @ 100 MHz"
+		(property "Description" "Ferrite bead"
 			(at 187.96 36.83 0)
 			(effects
@@
 			)
 		)
-		(property "Description" ""
+		(property "Description" "10uF Cap"
 			(at 138.43 40.64 0)
 			(effects
@@
 			)
 		)
-		(property "Digikey" "  2679-AGC1206X6S250-106KXETR-ND"
+		(property "Digikey" "1276-1804-1-ND"
 			(at 138.43 40.64 0)
 			(effects
@@
 		(unit 1)
 		(exclude_from_sim no)
-		(in_bom yes)
+		(in_bom no)
 		(on_board yes)
 		(dnp no)
@@
 			)
 		)
-		(property "Description" ""
+		(property "Description" "10k Res"
 			(at 31.75 62.23 0)
 			(effects
@@
 			)
 		)
-		(property "Description" ""
+		(property "Description" "100nF Cap"
 			(at 96.52 40.64 0)
 			(effects
@@
 			)
 		)
-		(property "Description" ""
+		(property "Description" "100nF Cap"
 			(at 106.68 40.64 0)
 			(effects
@@
 			)
 		)
-		(property "Description" ""
+		(property "Description" "10k Res"
 			(at 45.72 101.6 0)
 			(effects
@@
 			)
 		)
-		(property "Description" ""
+		(property "Description" "16pF Cap"
 			(at 30.48 137.16 0)
 			(effects
@@
 			)
 		)
-		(property "Description" ""
+		(property "Description" "1uF Cap"
 			(at 196.85 40.64 0)
 			(effects
@@
 			)
 		)
-		(property "Description" ""
+		(property "Description" "1uF Cap"
 			(at 176.53 40.64 0)
 			(effects
@@
 			)
 		)
-		(property "Description" ""
+		(property "Description" "100nF Cap"
 			(at 116.84 40.64 0)
 			(effects
@@
 			)
 		)
-		(property "Description" ""
+		(property "Description" "10o Res"
 			(at 53.34 128.27 0)
 			(effects
@@
 			)
 		)
-		(property "Description" ""
+		(property "Description" "10nF Cap"
 			(at 167.64 40.64 0)
 			(effects
@@
 		(unit 1)
 		(exclude_from_sim no)
-		(in_bom yes)
+		(in_bom no)
 		(on_board yes)
 		(dnp no)
@@
 		(unit 1)
 		(exclude_from_sim no)
-		(in_bom yes)
+		(in_bom no)
 		(on_board yes)
 		(dnp no)
@@
 			)
 		)
-		(property "Description" ""
+		(property "Description" "100nF Cap"
 			(at 115.57 58.42 0)
 			(effects
@@
 			)
 		)
-		(property "Description" ""
+		(property "Description" "100nF Cap"
 			(at 86.36 40.64 0)
 			(effects
@@
 			)
 		)
-		(property "Description" "406C35D08M00000"
+		(property "Description" "8MHz Cristal"
 			(at 38.1 128.27 0)
 			(effects
@@
 			)
 		)
-		(property "Digikey" "CTX853CT-ND"
+		(property "Digikey" "110-406C35D08M00000CT-ND"
 			(at 38.1 128.27 0)
 			(effects
@@
 			)
 		)
-		(property "Description" ""
+		(property "Description" "100nF Cap"
 			(at 127 40.64 0)
 			(effects
@@
 			)
 		)
-		(property "Description" ""
+		(property "Description" "10k Res"
 			(at 41.91 62.23 0)
 			(effects
