File: ReceiverRF/receiverKiCad/regulateurs.kicad_sch (KiCad schematic)
At the start: 15 parts, among them SW5 SW_SPST, U2 NCV5501DT33RKG, U3 NJM2882F05-TE1

Commit message: correction mineure, logo Idefix, commande PCBWAY
Parts:
- PWR_C1: value 10u -> 10uF; Digikey (none) -> 2679-AGC1206X6S250-106KXETR-ND
- PWR_C2: value 4.7u -> 4.7uF; Digikey (none) -> 4713-GMC10X7R475K10NTCT-ND
- PWR_C3: value 1u -> 1uF; Digikey (none) -> 2679-AGC0603X7R250-105KXPTR-ND
- PWR_C4: value 100n -> 100nF; Digikey (none) -> 2679-AGC0402X7R500-104KNPTR-ND
- PWR_C5: value 10n -> 10nF; Digikey (none) -> 2679-AGC0402X7R500-103KNPTR-ND
- PWR_D1, PWR_D2: value Rouge -> LTST-C190EKT; Digikey (none) -> 160-1182-1-ND
- PWR_R1, PWR_R2, PWR_R3, PWR_R4: value 145 -> 145R; Digikey (none) -> 2019-RN73H2BTTD1450F100CT-ND
- U2: Digikey (none) -> NCV5501DT33RKGOSCT-ND
- U3: Digikey (none) -> 2129-NJM2882F05-TE1CT-ND
Changed lines of the file:
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@@
 			)
 		)
-		(property "Value" "145"
+		(property "Value" "145R"
 			(at 78.74 73.66 0)
 			(effects
@@
 		)
 		(property "Description" ""
+			(at 76.2 72.39 0)
+			(effects
+				(font
+					(size 1.27 1.27)
+				)
+				(hide yes)
+			)
+		)
+		(property "Digikey" "2019-RN73H2BTTD1450F100CT-ND"
 			(at 76.2 72.39 0)
 			(effects
@@
 			)
 		)
-		(property "Value" "145"
+		(property "Value" "145R"
 			(at 219.71 96.52 0)
 			(effects
@@
 			)
 		)
+		(property "Digikey" "2019-RN73H2BTTD1450F100CT-ND"
+			(at 217.17 95.25 0)
+			(effects
+				(font
+					(size 1.27 1.27)
+				)
+				(hide yes)
+			)
+		)
 		(pin "1"
 		)
@@
 			)
 		)
-		(property "Value" "1u"
+		(property "Value" "1uF"
 			(at 204.47 87.63 0)
 			(effects
@@
 		)
 		(property "Description" ""
+			(at 201.93 86.36 0)
+			(effects
+				(font
+					(size 1.27 1.27)
+				)
+				(hide yes)
+			)
+		)
+		(property "Digikey" "  2679-AGC0603X7R250-105KXPTR-ND"
 			(at 201.93 86.36 0)
 			(effects
@@
 			)
 		)
-		(property "Value" "145"
+		(property "Value" "145R"
 			(at 210.82 77.47 90)
 			(effects
@@
 		)
 		(property "Description" ""
+			(at 210.82 81.28 0)
+			(effects
+				(font
+					(size 1.27 1.27)
+				)
+				(hide yes)
+			)
+		)
+		(property "Digikey" "2019-RN73H2BTTD1450F100CT-ND"
 			(at 210.82 81.28 0)
 			(effects
@@
 			)
 		)
+		(property "Digikey" ""
+			(at 53.34 33.02 0)
+			(effects
+				(font
+					(size 1.27 1.27)
+				)
+				(hide yes)
+			)
+		)
 		(pin "2"
 		)
@@
 			)
 		)
+		(property "Digikey" "2129-NJM2882F05-TE1CT-ND"
+			(at 134.62 81.28 0)
+			(effects
+				(font
+					(size 1.27 1.27)
+				)
+				(hide yes)
+			)
+		)
 		(pin "1"
 		)
@@
 			)
 		)
-		(property "Value" "4.7u"
+		(property "Value" "4.7uF"
 			(at 66.294 74.93 0)
 			(effects
@@
 		)
 		(property "Description" ""
+			(at 63.5 73.66 0)
+			(effects
+				(font
+					(size 1.27 1.27)
+				)
+				(hide yes)
+			)
+		)
+		(property "Digikey" "4713-GMC10X7R475K10NTCT-ND"
 			(at 63.5 73.66 0)
 			(effects
@@
 			)
 		)
-		(property "Value" "10n"
+		(property "Value" "10nF"
 			(at 193.04 97.79 0)
 			(effects
@@
 		)
 		(property "Description" ""
+			(at 190.5 96.52 0)
+			(effects
+				(font
+					(size 1.27 1.27)
+				)
+				(hide yes)
+			)
+		)
+		(property "Digikey" "  2679-AGC0402X7R500-103KNPTR-ND"
 			(at 190.5 96.52 0)
 			(effects
@@
 			)
 		)
+		(property "Digikey" ""
+			(at 38.1 33.02 0)
+			(effects
+				(font
+					(size 1.27 1.27)
+				)
+				(hide yes)
+			)
+		)
 		(pin "1"
 		)
@@
 			)
 		)
-		(property "Value" "100n"
+		(property "Value" "100nF"
 			(at 124.46 95.25 0)
 			(effects
@@
 		)
 		(property "Description" ""
+			(at 120.65 93.98 0)
+			(effects
+				(font
+					(size 1.27 1.27)
+				)
+				(hide yes)
+			)
+		)
+		(property "Digikey" "2679-AGC0402X7R500-104KNPTR-ND"
 			(at 120.65 93.98 0)
 			(effects
@@
 			)
 		)
-		(property "Value" "145"
+		(property "Value" "145R"
 			(at 219.71 87.63 0)
 			(effects
@@
 		)
 		(property "Description" ""
+			(at 217.17 86.36 0)
+			(effects
+				(font
+					(size 1.27 1.27)
+				)
+				(hide yes)
+			)
+		)
+		(property "Digikey" "2019-RN73H2BTTD1450F100CT-ND"
 			(at 217.17 86.36 0)
 			(effects
@@
 			)
 		)
-		(property "Value" "Rouge"
+		(property "Value" "LTST-C190EKT"
 			(at 78.74 82.55 0)
 			(effects
@@
 		)
 		(property "Description" ""
+			(at 76.2 81.28 0)
+			(effects
+				(font
+					(size 1.27 1.27)
+				)
+				(hide yes)
+			)
+		)
+		(property "Digikey" "160-1182-1-ND"
 			(at 76.2 81.28 0)
 			(effects
@@
 			)
 		)
-		(property "Value" "10u"
+		(property "Value" "10uF"
 			(at 37.084 74.676 0)
 			(effects
@@
 		)
 		(property "Description" ""
+			(at 34.29 73.66 0)
+			(effects
+				(font
+					(size 1.27 1.27)
+				)
+				(hide yes)
+			)
+		)
+		(property "Digikey" "  2679-AGC1206X6S250-106KXETR-ND"
 			(at 34.29 73.66 0)
 			(effects
@@
 			)
 		)
+		(property "Digikey" "NCV5501DT33RKGOSCT-ND "
+			(at 48.26 109.22 0)
+			(effects
+				(font
+					(size 1.27 1.27)
+				)
+				(hide yes)
+			)
+		)
 		(pin "1"
 		)
@@
 			)
 		)
-		(property "Value" "Rouge"
+		(property "Value" "LTST-C190EKT"
 			(at 219.71 104.14 0)
 			(effects
@@
 			(at 217.17 104.14 0)
 			(effects
+				(font
+					(size 1.27 1.27)
+				)
+				(hide yes)
+			)
+		)
+		(property "Digikey" "160-1182-1-ND"
+			(at 217.17 104.14 0)
+			(effects
